Commit message: c3_support: cleaned manifest, build script and deleted backups.

File: epson_c3_support/urdf/c3_macro.xacro (robot description, xacro)
@@ -10,5 +10,5 @@
         </geometry>
         <material name="">
-       	 <color rgba="1 1 1 1" />
+       	  <color rgba="1 1 1 1" />
       	</material>
       </visual>
@@ -27,5 +27,5 @@
         </geometry>
         <material name="">
-       	 <color rgba="1 1 1 1" />
+       	  <color rgba="1 1 1 1" />
       	</material>
       </visual>
@@ -44,5 +44,5 @@
         </geometry>
         <material name="">
-       	 <color rgba="1 1 1 1" />
+       	  <color rgba="1 1 1 1" />
       	</material>
       </visual>
@@ -61,5 +61,5 @@
         </geometry>
         <material name="">
-       	 <color rgba="1 1 1 1" />
+       	  <color rgba="1 1 1 1" />
       	</material>
       </visual>
@@ -78,5 +78,5 @@
         </geometry>
         <material name="">
-       	 <color rgba="1 1 1 1" />
+       	  <color rgba="1 1 1 1" />
       	</material>
       </visual>
@@ -95,5 +95,5 @@
         </geometry>
         <material name="">
-       	 <color rgba="1 1 1 1" />
+       	  <color rgba="1 1 1 1" />
       	</material>
       </visual>
@@ -112,5 +112,5 @@
         </geometry>
         <material name="">
-       	 <color rgba="1 1 1 1" />
+       	  <color rgba="1 1 1 1" />
       	</material>
       </visual>
@@ -129,5 +129,5 @@
       <child link="${prefix}link_1"/>
       <axis xyz="0 0 1"/>
-      <limit lower="-2.9671" upper="2.9671" effort="0" velocity="0"/>
+      <limit lower="-2.9671" upper="2.9671" effort="0" velocity="7.85"/>
     </joint>
     <joint name="${prefix}joint_2" type="revolute">
@@ -136,5 +136,5 @@
       <child link="${prefix}link_2"/>
       <axis xyz="1 0 0"/>
-      <limit lower="-2.7925" upper="1.1345" effort="0" velocity="0"/>
+      <limit lower="-2.7925" upper="1.1345" effort="0" velocity="7.85"/>
     </joint>
     <joint name="${prefix}joint_3" type="revolute">
@@ -143,5 +143,5 @@
       <child link="${prefix}link_3"/>
       <axis xyz="1 0 0"/>
-      <limit lower="-0.8901" upper="3.9270" effort="0" velocity="0"/>
+      <limit lower="-0.8901" upper="3.9270" effort="0" velocity="8.97"/>
     </joint>
     <joint name="${prefix}joint_4" type="revolute">
@@ -150,5 +150,5 @@
       <child link="${prefix}link_4"/>
       <axis xyz="0 -1 0"/>
-      <limit lower="-3.4907" upper="3.4907" effort="0" velocity="0"/>
+      <limit lower="-3.4907" upper="3.4907" effort="0" velocity="9.65"/>
     </joint>
     <joint name="${prefix}joint_5" type="revolute">
@@ -157,5 +157,5 @@
       <child link="${prefix}link_5"/>
       <axis xyz="1 0 0"/>
-      <limit lower="-2.3562" upper="2.3562" effort="0" velocity="0"/>
+      <limit lower="-2.3562" upper="2.3562" effort="0" velocity="9.65"/>
     </joint>
     <joint name="${prefix}joint_6" type="revolute">
@@ -164,5 +164,5 @@
       <child link="${prefix}link_6"/>
       <axis xyz="0 0 -1"/>
-      <limit lower="-6.2832" upper="6.2832" effort="0" velocity="0"/>
+      <limit lower="-6.2832" upper="6.2832" effort="0" velocity="12,56"/>
     </joint>
     <joint name="${prefix}joint_6-tool0" type="fixed">
@@ -170,4 +170,5 @@
       <parent link="${prefix}link_6"/>
       <child link="${prefix}tool0"/>
+      <axis xyz="0 0 0" />
     </joint>
     <!-- ROS base_link to Epson World Coordinates transform -->

Commit message: c3_support: use dots as decimal mark.

File: epson_c3_support/urdf/c3_macro.xacro (robot description, xacro)
@@ -164,5 +164,5 @@
       <child link="${prefix}link_6"/>
       <axis xyz="0 0 -1"/>
-      <limit lower="-6.2832" upper="6.2832" effort="0" velocity="12,56"/>
+      <limit lower="-6.2832" upper="6.2832" effort="0" velocity="12.56"/>
     </joint>
     <joint name="${prefix}joint_6-tool0" type="fixed">

Commit message: c3_support: fix xacro macro indent.

File: epson_c3_support/urdf/c3_macro.xacro (robot description, xacro)
@@ -10,6 +10,6 @@
         </geometry>
         <material name="">
-       	  <color rgba="1 1 1 1" />
-      	</material>
+          <color rgba="1 1 1 1" />
+        </material>
       </visual>
       <collision>
@@ -27,6 +27,6 @@
         </geometry>
         <material name="">
-       	  <color rgba="1 1 1 1" />
-      	</material>
+          <color rgba="1 1 1 1" />
+        </material>
       </visual>
       <collision>
@@ -44,6 +44,6 @@
         </geometry>
         <material name="">
-       	  <color rgba="1 1 1 1" />
-      	</material>
+          <color rgba="1 1 1 1" />
+        </material>
       </visual>
       <collision>
@@ -61,6 +61,6 @@
         </geometry>
         <material name="">
-       	  <color rgba="1 1 1 1" />
-      	</material>
+          <color rgba="1 1 1 1" />
+        </material>
       </visual>
       <collision>
@@ -78,6 +78,6 @@
         </geometry>
         <material name="">
-       	  <color rgba="1 1 1 1" />
-      	</material>
+          <color rgba="1 1 1 1" />
+        </material>
       </visual>
       <collision>
@@ -95,6 +95,6 @@
         </geometry>
         <material name="">
-       	  <color rgba="1 1 1 1" />
-      	</material>
+          <color rgba="1 1 1 1" />
+        </material>
       </visual>
       <collision>
@@ -112,6 +112,6 @@
         </geometry>
         <material name="">
-       	  <color rgba="1 1 1 1" />
-      	</material>
+          <color rgba="1 1 1 1" />
+        </material>
       </visual>
       <collision>

Commit message: c3_support: scale & transform C3 meshes.
This is a temporary fix until meshes have been properly scaled and
their origins have been corrected.

File: epson_c3_support/urdf/c3_macro.xacro (robot description, xacro)
@@ -7,5 +7,5 @@
         <origin xyz="0 0 0" rpy="0 0 0"/>
         <geometry>
-          <mesh filename="package://epson_c3_support/meshes/c3/visual/base_link.stl"/>
+          <mesh filename="package://epson_c3_support/meshes/c3/visual/base_link.stl" scale="0.001 0.001 0.001" />
         </geometry>
         <material name="">
@@ -16,5 +16,5 @@
         <origin xyz="0 0 0" rpy="0 0 0"/>
         <geometry>
-          <mesh filename="package://epson_c3_support/meshes/c3/collision/base_link.stl"/>
+          <mesh filename="package://epson_c3_support/meshes/c3/collision/base_link.stl" scale="0.001 0.001 0.001" />
         </geometry>
       </collision>
@@ -22,7 +22,7 @@
     <link name="${prefix}link_1">
       <visual>
-        <origin xyz="0 0 0" rpy="0 0 0"/>
+        <origin xyz="0 0 -0.1965" rpy="0 0 0"/>
         <geometry>
-          <mesh filename="package://epson_c3_support/meshes/c3/visual/link_1.stl"/>
+          <mesh filename="package://epson_c3_support/meshes/c3/visual/link_1.stl" scale="0.001 0.001 0.001" />
         </geometry>
         <material name="">
@@ -31,7 +31,7 @@
       </visual>
       <collision>
-        <origin xyz="0 0 0" rpy="0 0 0"/>
+        <origin xyz="0 0 -0.1965" rpy="0 0 0"/>
         <geometry>
-          <mesh filename="package://epson_c3_support/meshes/c3/collision/link_1.stl"/>
+          <mesh filename="package://epson_c3_support/meshes/c3/collision/link_1.stl" scale="0.001 0.001 0.001" />
         </geometry>
       </collision>
@@ -39,7 +39,7 @@
     <link name="${prefix}link_2">
       <visual>
-        <origin xyz="0 0 0" rpy="0 0 0"/>
+        <origin xyz="0 -0.1 -0.320" rpy="0 0 0"/>
         <geometry>
-          <mesh filename="package://epson_c3_support/meshes/c3/visual/link_2.stl"/>
+          <mesh filename="package://epson_c3_support/meshes/c3/visual/link_2.stl" scale="0.001 0.001 0.001" />
         </geometry>
         <material name="">
@@ -48,7 +48,7 @@
       </visual>
       <collision>
-        <origin xyz="0 0 0" rpy="0 0 0"/>
+        <origin xyz="0 -0.1 -0.320" rpy="0 0 0"/>
         <geometry>
-          <mesh filename="package://epson_c3_support/meshes/c3/collision/link_2.stl"/>
+          <mesh filename="package://epson_c3_support/meshes/c3/collision/link_2.stl" scale="0.001 0.001 0.001" />
         </geometry>
       </collision>
@@ -56,7 +56,7 @@
     <link name="${prefix}link_3">
       <visual>
-        <origin xyz="0 0 0" rpy="0 0 0"/>
+        <origin xyz="0 -0.1 -0.57" rpy="0 0 0"/>
         <geometry>
-          <mesh filename="package://epson_c3_support/meshes/c3/visual/link_3.stl"/>
+          <mesh filename="package://epson_c3_support/meshes/c3/visual/link_3.stl" scale="0.001 0.001 0.001" />
         </geometry>
         <material name="">
@@ -65,7 +65,7 @@
       </visual>
       <collision>
-        <origin xyz="0 0 0" rpy="0 0 0"/>
+        <origin xyz="0 -0.1 -0.57" rpy="0 0 0"/>
         <geometry>
-          <mesh filename="package://epson_c3_support/meshes/c3/collision/link_3.stl"/>
+          <mesh filename="package://epson_c3_support/meshes/c3/collision/link_3.stl" scale="0.001 0.001 0.001" />
         </geometry>
       </collision>
@@ -73,7 +73,7 @@
     <link name="${prefix}link_4">
       <visual>
-        <origin xyz="0 0 0" rpy="0 0 0"/>
+        <origin xyz="0 -0.1 -0.57" rpy="0 0 0"/>
         <geometry>
-          <mesh filename="package://epson_c3_support/meshes/c3/visual/link_4.stl"/>
+          <mesh filename="package://epson_c3_support/meshes/c3/visual/link_4.stl" scale="0.001 0.001 0.001" />
         </geometry>
         <material name="">
@@ -82,7 +82,7 @@
       </visual>
       <collision>
-        <origin xyz="0 0 0" rpy="0 0 0"/>
+        <origin xyz="0 -0.1 -0.57" rpy="0 0 0"/>
         <geometry>
-          <mesh filename="package://epson_c3_support/meshes/c3/collision/link_4.stl"/>
+          <mesh filename="package://epson_c3_support/meshes/c3/collision/link_4.stl" scale="0.001 0.001 0.001" />
         </geometry>
       </collision>
@@ -90,7 +90,7 @@
     <link name="${prefix}link_5">
       <visual>
-        <origin xyz="0 0 0" rpy="0 0 0"/>
+        <origin xyz="0 -0.35 -0.57" rpy="0 0 0"/>
         <geometry>
-          <mesh filename="package://epson_c3_support/meshes/c3/visual/link_5.stl"/>
+          <mesh filename="package://epson_c3_support/meshes/c3/visual/link_5.stl" scale="0.001 0.001 0.001" />
         </geometry>
         <material name="">
@@ -99,7 +99,7 @@
       </visual>
       <collision>
-        <origin xyz="0 0 0" rpy="0 0 0"/>
+        <origin xyz="0 -0.35 -0.57" rpy="0 0 0"/>
         <geometry>
-          <mesh filename="package://epson_c3_support/meshes/c3/collision/link_5.stl"/>
+          <mesh filename="package://epson_c3_support/meshes/c3/collision/link_5.stl" scale="0.001 0.001 0.001" />
         </geometry>
       </collision>
@@ -107,7 +107,7 @@
     <link name="${prefix}link_6">
       <visual>
-        <origin xyz="0 0 0" rpy="0 0 0"/>
+        <origin xyz="-0.57 0 -0.41" rpy="1.570796326 0 1.570796326"/>
         <geometry>
-          <mesh filename="package://epson_c3_support/meshes/c3/visual/link_6.stl"/>
+          <mesh filename="package://epson_c3_support/meshes/c3/visual/link_6.stl" scale="0.001 0.001 0.001" />
         </geometry>
         <material name="">
@@ -116,7 +116,7 @@
       </visual>
       <collision>
-        <origin xyz="0 0 0" rpy="0 0 0"/>
+        <origin xyz="-0.57 0 -0.41" rpy="1.570796326 0 1.570796326"/>
         <geometry>
-          <mesh filename="package://epson_c3_support/meshes/c3/collision/link_6.stl"/>
+          <mesh filename="package://epson_c3_support/meshes/c3/collision/link_6.stl" scale="0.001 0.001 0.001" />
         </geometry>
       </collision>

Commit message: c3_support: correct pose of link_6 (and meshes).

File: epson_c3_support/urdf/c3_macro.xacro (robot description, xacro)
@@ -107,5 +107,5 @@
     <link name="${prefix}link_6">
       <visual>
-        <origin xyz="-0.57 0 -0.41" rpy="1.570796326 0 1.570796326"/>
+        <origin xyz="0 -0.41 -0.57" rpy="0 0 0"/>
         <geometry>
           <mesh filename="package://epson_c3_support/meshes/c3/visual/link_6.stl" scale="0.001 0.001 0.001" />
@@ -116,5 +116,5 @@
       </visual>
       <collision>
-        <origin xyz="-0.57 0 -0.41" rpy="1.570796326 0 1.570796326"/>
+        <origin xyz="0 -0.41 -0.57" rpy="0 0 0"/>
         <geometry>
           <mesh filename="package://epson_c3_support/meshes/c3/collision/link_6.stl" scale="0.001 0.001 0.001" />
@@ -160,12 +160,12 @@
     </joint>
     <joint name="${prefix}joint_6" type="revolute">
-      <origin xyz="0 0.06 0" rpy="-1.570796326 -1.570796326 0"/>
+      <origin xyz="0 0.06 0" rpy="0 0 0"/>
       <parent link="${prefix}link_5"/>
       <child link="${prefix}link_6"/>
-      <axis xyz="0 0 -1"/>
+      <axis xyz="0 -1 0"/>
       <limit lower="-6.2832" upper="6.2832" effort="0" velocity="12.56"/>
     </joint>
     <joint name="${prefix}joint_6-tool0" type="fixed">
-      <origin xyz="0 0 0.005" rpy="0 0 0.785398163" />
+      <origin xyz="0 0.005 0" rpy="-1.570796326 -1.570796326 0" />
       <parent link="${prefix}link_6"/>
       <child link="${prefix}tool0"/>

Commit message: c3_support: correct 'base' link origin.
Epson has world coordinate origin at "intersection of robot base and
joint 1 axis".

File: epson_c3_support/urdf/c3_macro.xacro (robot description, xacro)
@@ -175,5 +175,5 @@
     <link name="${prefix}base" />
     <joint name="${prefix}base_link-base" type="fixed">
-      <origin xyz="0 0 0.1965" rpy="0 0 0"/>
+      <origin xyz="0 0 0" rpy="0 0 0"/>
       <parent link="${prefix}base_link"/>
       <child link="${prefix}base"/>

Commit message: c3_support: correct tool0 pose.

File: epson_c3_support/urdf/c3_macro.xacro (robot description, xacro)
@@ -167,5 +167,5 @@
     </joint>
     <joint name="${prefix}joint_6-tool0" type="fixed">
-      <origin xyz="0 0.005 0" rpy="-1.570796326 -1.570796326 0" />
+      <origin xyz="0 0.005 0" rpy="-1.570796327 -1.570796327 0" />
       <parent link="${prefix}link_6"/>
       <child link="${prefix}tool0"/>
