Commit message: update support package

File: epson_c3_support/urdf/c3a601s.xacro (robot description, xacro)
@@ -1,5 +1,5 @@
 <?xml version="1.0" ?>
 <robot name="epson_c3a601s" xmlns:xacro="http://ros.org/wiki/xacro">
-  <xacro:include filename="$(find epson_c3a601s_support)/urdf/c3a601s_macro.xacro"/>
+  <xacro:include filename="$(find epson_c3_support)/urdf/c3a601s_macro.xacro"/>
   <xacro:epson_c3a601s prefix=""/>
 </robot>

File: epson_c3_support/urdf/c3a601s_macro.xacro (robot description, xacro)
@@ -7,5 +7,5 @@
         <origin xyz="0 0 0" rpy="0 0 -1.570796326"/>
         <geometry>
-          <mesh filename="package://epson_c3a601s_support/meshes/c3a601s/visual/base_link.stl"/>
+          <mesh filename="package://epson_c3_support/meshes/c3a601s/visual/base_link.stl"/>
         </geometry>
         <material name="">
@@ -16,5 +16,5 @@
         <origin xyz="0 0 0" rpy="0 0 -1.570796326"/>
         <geometry>
-          <mesh filename="package://epson_c3a601s_support/meshes/c3a601s/collision/base_link.stl"/>
+          <mesh filename="package://epson_c3_support/meshes/c3a601s/collision/base_link.stl"/>
         </geometry>
       </collision>
@@ -24,5 +24,5 @@
         <origin xyz="0 0 0" rpy="0 0 -1.570796326"/>
         <geometry>
-          <mesh filename="package://epson_c3a601s_support/meshes/c3a601s/visual/link_1.stl"/>
+          <mesh filename="package://epson_c3_support/meshes/c3a601s/visual/link_1.stl"/>
         </geometry>
         <material name="">
@@ -33,5 +33,5 @@
         <origin xyz="0 0 0" rpy="0 0 -1.570796326"/>
         <geometry>
-          <mesh filename="package://epson_c3a601s_support/meshes/c3a601s/collision/link_1.stl"/>
+          <mesh filename="package://epson_c3_support/meshes/c3a601s/collision/link_1.stl"/>
         </geometry>
       </collision>
@@ -41,5 +41,5 @@
         <origin xyz="0 0 0" rpy="0 0 -1.570796326"/>
         <geometry>
-          <mesh filename="package://epson_c3a601s_support/meshes/c3a601s/visual/link_2.stl"/>
+          <mesh filename="package://epson_c3_support/meshes/c3a601s/visual/link_2.stl"/>
         </geometry>
         <material name="">
@@ -50,5 +50,5 @@
         <origin xyz="0 0 0" rpy="0 0 -1.570796326"/>
         <geometry>
-          <mesh filename="package://epson_c3a601s_support/meshes/c3a601s/collision/link_2.stl"/>
+          <mesh filename="package://epson_c3_support/meshes/c3a601s/collision/link_2.stl"/>
         </geometry>
       </collision>
@@ -58,5 +58,5 @@
         <origin xyz="0 0 0" rpy="0 0 -1.570796326"/>
         <geometry>
-          <mesh filename="package://epson_c3a601s_support/meshes/c3a601s/visual/link_3.stl"/>
+          <mesh filename="package://epson_c3_support/meshes/c3a601s/visual/link_3.stl"/>
         </geometry>
         <material name="">
@@ -67,5 +67,5 @@
         <origin xyz="0 0 0" rpy="0 0 -1.570796326"/>
         <geometry>
-          <mesh filename="package://epson_c3a601s_support/meshes/c3a601s/collision/link_3.stl"/>
+          <mesh filename="package://epson_c3_support/meshes/c3a601s/collision/link_3.stl"/>
         </geometry>
       </collision>
@@ -75,5 +75,5 @@
         <origin xyz="0 0 0" rpy="0 0 -1.570796326"/>
         <geometry>
-          <mesh filename="package://epson_c3a601s_support/meshes/c3a601s/visual/link_4.stl"/>
+          <mesh filename="package://epson_c3_support/meshes/c3a601s/visual/link_4.stl"/>
         </geometry>
         <material name="">
@@ -84,5 +84,5 @@
         <origin xyz="0 0 0" rpy="0 0 -1.570796326"/>
         <geometry>
-          <mesh filename="package://epson_c3a601s_support/meshes/c3a601s/collision/link_4.stl"/>
+          <mesh filename="package://epson_c3_support/meshes/c3a601s/collision/link_4.stl"/>
         </geometry>
       </collision>
@@ -92,5 +92,5 @@
         <origin xyz="0 0 0" rpy="0 0 -1.570796326"/>
         <geometry>
-          <mesh filename="package://epson_c3a601s_support/meshes/c3a601s/visual/link_5.stl"/>
+          <mesh filename="package://epson_c3_support/meshes/c3a601s/visual/link_5.stl"/>
         </geometry>
         <material name="">
@@ -101,5 +101,5 @@
         <origin xyz="0 0 0" rpy="0 0 -1.570796326"/>
         <geometry>
-          <mesh filename="package://epson_c3a601s_support/meshes/c3a601s/collision/link_5.stl"/>
+          <mesh filename="package://epson_c3_support/meshes/c3a601s/collision/link_5.stl"/>
         </geometry>
       </collision>
@@ -109,5 +109,5 @@
         <origin xyz="0 0 0" rpy="0 0 -1.570796326"/>
         <geometry>
-          <mesh filename="package://epson_c3a601s_support/meshes/c3a601s/visual/link_6.stl"/>
+          <mesh filename="package://epson_c3_support/meshes/c3a601s/visual/link_6.stl"/>
         </geometry>
         <material name="">
@@ -118,5 +118,5 @@
         <origin xyz="0 0 0" rpy="0 0 -1.570796326"/>
         <geometry>
-          <mesh filename="package://epson_c3a601s_support/meshes/c3a601s/collision/link_6.stl"/>
+          <mesh filename="package://epson_c3_support/meshes/c3a601s/collision/link_6.stl"/>
         </geometry>
       </collision>
